File: pcb/mate-net-monitor.sch (KiCad schematic (older format))
At the start: 1 part

Commit message: schematic P1 Draft 1
Parts:
- added C? (x2): 1uF, symbol Device:C_Small
- added C?: 470nF, symbol Device:C_Small
- added C?: 1nF, symbol Device:C_Small
- added C?: 12nF, symbol Device:C_Small
- added C?: 1.3nF, symbol Device:C_Small
- added C? (x2): 47uF, symbol Device:C_Small
- added C?: ?uF, symbol Device:C_Small
- added D?: D_Schottky_Small_ALT, symbol Device:D_Schottky_Small_ALT
- added D? (x3): D_Small_ALT, symbol Device:D_Small_ALT
- added D? (x3): Green, symbol Device:LED_Small_ALT
- added D?: Yellow, symbol Device:LED_Small_ALT
- added D?: Red, symbol Device:LED_Small_ALT
- added H?: Enclosure_WM032C, symbol mate-net-monitor-special:Enclosure_WM032C
- added H?: Light_Pipe_3x1_7511B11, symbol mate-net-monitor-special:Light_Pipe_3x1_7511B11
- added H? (x2): M3, symbol Mechanical:MountingHole_Pad
- added J?: RJHSE-5081, symbol Connector:RJ45_LED
- added J? (x2): 6P6C, symbol Connector:6P6C
- added J?: Conn_02x04_Odd_Even, symbol Connector_Generic:Conn_02x04_Odd_Even
- added L?: 68uH 100mOhm, symbol Device:L
- added Q?: Si2337DS, symbol Device:Q_PMOS_GSD
- added R?: 133k, symbol Device:R_Small
- added R?: 845, symbol Device:R_Small
- added R?: 10m 0.5W, symbol Device:R_Small
- added R?: 80.6k, symbol Device:R_Small
- added R? (x5): 10k, symbol Device:R_Small
- added R?: 3.32k, symbol Device:R_Small
- added R? (x3): 4.7k, symbol Device:R_Small
- added R? (x6): 1k, symbol Device:R_Small
- added R?: 0, symbol Device:R_Small
- added R? (x4): 22, symbol Device:R_Small
- added R?: 0-DNP, symbol Device:R_Small
- added U? (x2): TLP185, Package_SO:SOIC-4_4.55x3.7mm_P2.54mm, symbol Isolator:TLP185
- added U?: LM5085MY, Package_SO:MSOP-8-1EP_3x3mm_P0.65mm_EP1.73x1.85mm_ThermalVias, symbol mate-net-monitor-special:LM5085MY
- added U?: MAX3485, symbol Interface_UART:MAX3485
Connections:
- net labels added: +3.3V, +3V3, +5V, +BATT, CONN_ADC1, CONN_ADC2, CONN_ADC3, CONN_ADC4, GND, MAG_NET_A, MAG_NET_B, MAG_NET_GND, MAG_NET_GND_K, MAG_NET_P14V, MAG_NET_P14V_K, MATE_NET_K, MATE_NET_RXD, MATE_NET_RXD_K, MATE_NET_TXD, P3V3_K, P5V_ISEN, P5V_K, PBATT_CONN, PBATT_K, PB_ADC1, PB_ADC2, PB_ADC3, PB_ADC4, PB_D2, PB_D2_R, PB_D3, PB_PWM2, PB_UART1_RX, PB_UART1_TX, PB_UART2_RX, PB_UART2_TX
- wire segments 0 -> 242
- no-connect marks 0 -> 8
Other:
- note added: "1.1mA\n@ 14V"
- note added: "1.1mA\n@ 3.3V"
- note added: "From Inverter"
- note added: "Green"
- note added: "Green: Mag Net Ok\nYellow: Mag Net Traffic\nRed: Mag Net Flipped"
- note added: "MATE Net\nUART @ Vbatt\n9600 9n1"
- note added: "MATE Vbatt\n24V Sys: 16-28.4Vdc\n48V Sys: 32-56.8Vdc"
- note added: "Note: Not connecting\nMag Net GND due to\nrisk of 14V/GND short."
- note added: "To Remote"
- note added: "UART @ 3.3V\n9600 9n1"
- note added: "VinMin=16.0V\nVinMax=58.0V\nVout=5.0V\nIout=1.5A"
- note added: "Yellow"
- moved on the sheet: A?

Commit message: schematic P1 Draft 2 and footprints
Parts:
- added D1, D11, D2, D3: Vr=60V, Diode_SMD:D_SOD-123F, symbol Device:D_TVS_ALT
- added J3: Conn_02x02_Odd_Even, Connector_PinSocket_2.54mm:PinSocket_2x02_P2.54mm_Vertical, symbol Connector_Generic:Conn_02x02_Odd_Even
- added R11: 2.2k, Resistor_SMD:R_0805_2012Metric, symbol Device:R_Small
- added U2: TLP185, Package_SO:SOIC-4_4.55x3.7mm_P2.54mm, symbol Isolator:TLP185
- A1: renamed from A?; footprint (none) -> mate-net-monitor-special:Particle_Boron_1x16_1x12_P2.54mm
- C1, C2: renamed from C?; footprint (none) -> Capacitor_SMD:C_1210_3225Metric
- C3, C4, C5, C6: renamed from C?; footprint (none) -> Capacitor_SMD:C_0805_2012Metric
- C7, C8: renamed from C?; footprint (none) -> Capacitor_SMD:C_1206_3216Metric
- C9: renamed from C?; footprint (none) -> Capacitor_SMD:CP_Elec_4x4.5
- D10, D6, D7, D8, D9: renamed from D?; footprint (none) -> LED_SMD:LED_0603_1608Metric_Pad1.05x0.95mm_HandSolder
- D12, D13, D4, D5: renamed from D?; footprint (none) -> Diode_SMD:D_SMA
- H1: renamed from H?; footprint (none) -> mate-net-monitor-special:Enclosure_WM032C
- H2: renamed from H?; footprint (none) -> mate-net-monitor-special:Light_Pipe_3x1_7511B11
- H3, H4: renamed from H?; footprint (none) -> mate-net-monitor-special:MountingHole_3mm_Pad_Via_NoPTH
- J1: renamed from J?; footprint (none) -> mate-net-monitor-special:RJ45_Amphenol_RJHSE508X
- J2: renamed from J?; footprint (none) -> Connector_PinSocket_2.54mm:PinSocket_2x04_P2.54mm_Vertical
- J4, J5: renamed from J?; footprint (none) -> Connector_RJ:RJ12_Amphenol_54601
- L1: renamed from L?; footprint (none) -> Inductor_SMD:L_Bourns_SRR1210A
- Q1: renamed from Q?; footprint (none) -> Package_TO_SOT_SMD:SOT-23
- R1: renamed from R?; value 1k -> 33k; footprint (none) -> Resistor_SMD:R_0805_2012Metric
- R10, R15, R16, R17, R18, R19, R20, R21, R22, R23, R24, R25, R26, R3, R4, R7, R8, R9: renamed from R?; footprint (none) -> Resistor_SMD:R_0805_2012Metric
- R12, R13: renamed from R?; value 1k -> 2.2k; footprint (none) -> Resistor_SMD:R_0805_2012Metric
- R14: renamed from R?; footprint (none) -> Resistor_SMD:R_1206_3216Metric
- R2, R5, R6: renamed from R?; value 4.7k -> 33k; footprint (none) -> Resistor_SMD:R_0805_2012Metric
- U5: renamed from U?; footprint (none) -> Package_SO:SOIC-8_3.9x4.9mm_P1.27mm
- gave numbers to parts that had none: 3
Connections:
- net labels added: MAG_NET_GND_R, MAG_NET_P14V_R, MATE_NET_IND_A, MATE_NET_IND_R, PB_SCL, PB_SDA
- net labels removed: MATE_NET_K
- wire segments 242 -> 277
Other:
- note added: "1.4mA\n@ 48V"
- note added: "Blink traffic LED w/\nBoron PWM @ 5Hz"
- moved on the sheet: D9, R1, R22

Commit message: layout P1
Parts:
- removed J2: Conn_02x04_Odd_Even, Connector_PinSocket_2.54mm:PinSocket_2x04_P2.54mm_Vertical, symbol Connector_Generic:Conn_02x04_Odd_Even
- removed R15: 0, Resistor_SMD:R_0805_2012Metric, symbol Device:R_Small
- added J4: Conn_01x08, Connector_PinSocket_2.54mm:PinSocket_1x08_P2.54mm_Vertical, symbol Connector_Generic:Conn_01x08
- C9: value ?uF -> 180uF; footprint Capacitor_SMD:CP_Elec_4x4.5 -> Capacitor_SMD:CP_Elec_6.3x5.9
- R4, R7, R8, R9: value 22 -> 47k
- renumbered J4 to J1, J5 to J2, J1 to J5
Connections:
- net labels added: P5V_AC, P5V_ADJ, P5V_PGATE, P5V_SW, P5V_VCC, U5_EN
- wire segments 277 -> 278
- no-connect marks 8 -> 16
Other:
- note added: "1.1mA\n@ 56V\nlimiting\n"
- note added: "ADC Expansion for\nDC/AC Current"
- note added: "I2C Expansion for\nDC/AC Current"
- note added: "Int. Btn."
- note added: "Int. PU"
- note added: "Int.\nPU"
- note added: "from Boron"
- note added: "to Boron"
- moved on the sheet: R4, R7, R8, R9

Commit message: layout P1 schematic P1
review and fix circuits before fab
* fix Q1 D/S orientation
* fix J1/J2 labels to match pin usage
* add 3d models RJ45, RJ12, Boron, inductor
* new gerbers and pdfs
Parts:
- removed C9: 180uF, Capacitor_SMD:CP_Elec_6.3x5.9, symbol Device:C_Small
- added C9: 180uF, Capacitor_SMD:CP_Elec_6.3x5.9, symbol Device:CP1_Small
- added R27, R28: 4.7k-DNP, Resistor_SMD:R_0805_2012Metric, symbol Device:R_Small
- C1, C2: value 1uF -> 3.3uF
- D12, D13, D4, D5: Mfg (none) -> SMC Diode Solutions; Mfg PN (none) -> SK220ATR
- L1: Mfg (none) -> Bourns; Mfg PN (none) -> SRR1210-680M
- R3: value 133k -> 118k
- renumbered J2 to J1, J1 to J2
Connections:
- wire segments 278 -> 282
Other:
- moved on the sheet: J3
Changed lines of the file:
@@
 Sheet 1 1
 Title "Mate Net Monitor"
-Date "2021-08-22"
-Rev "P1 Draft 3"
+Date "2021-08-24"
+Rev "P1"
 Comp "Designed By: Ian Hartwig"
 Comment1 "Baseboard PCBA for MATE Net monitoring with a Particle Boron"
@@
 $EndComp
 $Comp
-L Connector:6P6C J2
+L Connector:6P6C J1
 U 1 1 61251B40
 P 9450 2700
-F 0 "J2" H 9507 3267 50  0000 C CNN
+F 0 "J1" H 9507 3267 50  0000 C CNN
 F 1 "6P6C" H 9507 3176 50  0000 C CNN
 F 2 "Connector_RJ:RJ12_Amphenol_54601" V 9450 2725 50  0001 C CNN
@@
 U 1 1 612771BC
 P 3400 6200
-F 0 "Q1" H 3604 6246 50  0000 L CNN
-F 1 "Si2337DS" H 3604 6155 50  0000 L CNN
+F 0 "Q1" H 3604 6154 50  0000 L CNN
+F 1 "Si2337DS" H 3604 6245 50  0000 L CNN
 F 2 "Package_TO_SOT_SMD:SOT-23" H 3600 6300 50  0001 C CNN
 F 3 "~" H 3400 6200 50  0001 C CNN
@@
 F 5 "SI2337DS-T1-E3" H 3400 6200 50  0001 C CNN "Mfg PN"
 	1    3400 6200
-	1    0    0    -1
+	1    0    0    1
 $EndComp
 $Comp
@@
 P 1100 6100
 F 0 "C2" H 1192 6146 50  0000 L CNN
-F 1 "1uF" H 1192 6055 50  0000 L CNN
+F 1 "3.3uF" H 1192 6055 50  0000 L CNN
 F 2 "Capacitor_SMD:C_1210_3225Metric" H 1100 6100 50  0001 C CNN
 F 3 "~" H 1100 6100 50  0001 C CNN
@@
 P 1550 6100
 F 0 "R3" H 1609 6146 50  0000 L CNN
-F 1 "133k" H 1609 6055 50  0000 L CNN
+F 1 "118k" H 1609 6055 50  0000 L CNN
 F 2 "Resistor_SMD:R_0805_2012Metric" H 1550 6100 50  0001 C CNN
 F 3 "~" H 1550 6100 50  0001 C CNN
@@
 F 2 "Diode_SMD:D_SMA" V 3500 6700 50  0001 C CNN
 F 3 "~" V 3500 6700 50  0001 C CNN
+F 4 "SMC Diode Solutions" V 3500 6700 50  0001 C CNN "Mfg"
+F 5 "SK220ATR" V 3500 6700 50  0001 C CNN "Mfg PN"
 	1    3500 6700
 	0    1    1    0
@@
 F 2 "Inductor_SMD:L_Bourns_SRR1210A" H 4500 6250 50  0001 C CNN
 F 3 "~" H 4500 6250 50  0001 C CNN
+F 4 "Bourns" V 4500 6250 50  0001 C CNN "Mfg"
+F 5 "SRR1210-680M" V 4500 6250 50  0001 C CNN "Mfg PN"
 	1    4500 6250
 	0    -1   -1   0
@@
 P 650 6100
 F 0 "C1" H 742 6146 50  0000 L CNN
-F 1 "1uF" H 742 6055 50  0000 L CNN
+F 1 "3.3uF" H 742 6055 50  0000 L CNN
 F 2 "Capacitor_SMD:C_1210_3225Metric" H 650 6100 50  0001 C CNN
 F 3 "~" H 650 6100 50  0001 C CNN
@@
 	2500 5250 2900 5250
 $Comp
-L Device:C_Small C9
-U 1 1 612E3C7C
-P 6550 6450
-F 0 "C9" H 6642 6496 50  0000 L CNN
-F 1 "180uF" H 6642 6405 50  0000 L CNN
-F 2 "Capacitor_SMD:CP_Elec_6.3x5.9" H 6550 6450 50  0001 C CNN
-F 3 "~" H 6550 6450 50  0001 C CNN
-	1    6550 6450
-	1    0    0    -1
-$EndComp
-$Comp
 L power:+5V #PWR0104
 U 1 1 612E7678
@@
 F 2 "Diode_SMD:D_SMA" V 1950 2950 50  0001 C CNN
 F 3 "~" V 1950 2950 50  0001 C CNN
+F 4 "SMC Diode Solutions" V 1950 2950 50  0001 C CNN "Mfg"
+F 5 "SK220ATR" V 1950 2950 50  0001 C CNN "Mfg PN"
 	1    1950 2950
 	0    1    1    0
@@
 Wire Wire Line
 	9450 4950 9450 4850
+Text Notes 9150 1250 0    50   ~ 0
+From Inverter
 Text Notes 9150 2350 0    50   ~ 0
-From Inverter
-Text Notes 9150 1250 0    50   ~ 0
 To Remote
 $Comp
-L Connector:6P6C J1
+L Connector:6P6C J2
 U 1 1 6122E1CC
 P 9450 1600
-F 0 "J1" H 9507 2167 50  0000 C CNN
+F 0 "J2" H 9507 2167 50  0000 C CNN
 F 1 "6P6C" H 9507 2076 50  0000 C CNN
 F 2 "Connector_RJ:RJ12_Amphenol_54601" V 9450 1625 50  0001 C CNN
@@
 F 2 "Diode_SMD:D_SMA" V 10600 1300 50  0001 C CNN
 F 3 "~" V 10600 1300 50  0001 C CNN
+F 4 "SMC Diode Solutions" V 10600 1300 50  0001 C CNN "Mfg"
+F 5 "SK220ATR" V 10600 1300 50  0001 C CNN "Mfg PN"
 	1    10600 1300
 	0    1    1    0
@@
 F 2 "Diode_SMD:D_SMA" V 10300 1300 50  0001 C CNN
 F 3 "~" V 10300 1300 50  0001 C CNN
+F 4 "SMC Diode Solutions" V 10300 1300 50  0001 C CNN "Mfg"
+F 5 "SK220ATR" V 10300 1300 50  0001 C CNN "Mfg PN"
 	1    10300 1300
 	0    1    1    0
@@
 L Connector_Generic:Conn_02x02_Odd_Even J3
 U 1 1 61B5AB24
-P 7000 4200
-F 0 "J3" H 7050 4417 50  0000 C CNN
-F 1 "Conn_02x02_Odd_Even" H 7050 4326 50  0000 C CNN
-F 2 "Connector_PinSocket_2.54mm:PinSocket_2x02_P2.54mm_Vertical" H 7000 4200 50  0001 C CNN
-F 3 "~" H 7000 4200 50  0001 C CNN
-	1    7000 4200
+P 6250 4450
+F 0 "J3" H 6300 4667 50  0000 C CNN
+F 1 "Conn_02x02_Odd_Even" H 6300 4576 50  0000 C CNN
+F 2 "Connector_PinSocket_2.54mm:PinSocket_2x02_P2.54mm_Vertical" H 6250 4450 50  0001 C CNN
+F 3 "~" H 6250 4450 50  0001 C CNN
+	1    6250 4450
 	1    0    0    -1
 $EndComp
@@
 L power:+3.3V #PWR0130
 U 1 1 61B5C87C
-P 6550 4100
-F 0 "#PWR0130" H 6550 3950 50  0001 C CNN
-F 1 "+3.3V" H 6565 4273 50  0000 C CNN
-F 2 "" H 6550 4100 50  0001 C CNN
-F 3 "" H 6550 4100 50  0001 C CNN
-	1    6550 4100
+P 5800 4350
+F 0 "#PWR0130" H 5800 4200 50  0001 C CNN
+F 1 "+3.3V" H 5815 4523 50  0000 C CNN
+F 2 "" H 5800 4350 50  0001 C CNN
+F 3 "" H 5800 4350 50  0001 C CNN
+	1    5800 4350
 	1    0    0    -1
 $EndComp
@@
 L power:GND #PWR0131
 U 1 1 61B5CDB8
-P 6550 4400
-F 0 "#PWR0131" H 6550 4150 50  0001 C CNN
-F 1 "GND" H 6555 4227 50  0000 C CNN
-F 2 "" H 6550 4400 50  0001 C CNN
-F 3 "" H 6550 4400 50  0001 C CNN
-	1    6550 4400
-	1    0    0    -1
-$EndComp
-Wire Wire Line
-	6550 4100 6550 4200
-Wire Wire Line
-	6550 4200 6800 4200
-Wire Wire Line
-	6550 4400 6550 4300
-Wire Wire Line
-	6550 4300 6800 4300
-Wire Wire Line
-	7300 4200 7750 4200
-Wire Wire Line
-	7750 4200 7750 3600
+P 5800 4650
+F 0 "#PWR0131" H 5800 4400 50  0001 C CNN
+F 1 "GND" H 5805 4477 50  0000 C CNN
+F 2 "" H 5800 4650 50  0001 C CNN
+F 3 "" H 5800 4650 50  0001 C CNN
+	1    5800 4650
+	1    0    0    -1
+$EndComp
+Wire Wire Line
+	5800 4350 5800 4450
+Wire Wire Line
+	5800 4450 6050 4450
+Wire Wire Line
+	5800 4650 5800 4550
+Wire Wire Line
+	5800 4550 6050 4550
+Wire Wire Line
+	6550 4450 6800 4450
+Wire Wire Line
+	7750 4450 7750 3600
 Wire Wire Line
 	7750 3600 7300 3600
 Wire Wire Line
-	7300 4300 7850 4300
-Wire Wire Line
-	7850 4300 7850 3450
+	6550 4550 7300 4550
+Wire Wire Line
+	7850 4550 7850 3450
 Wire Wire Line
 	7850 3450 7300 3450
@@
 Wire Wire Line
 	1250 1050 2550 1050
-Text Notes 6750 4600 0    50   ~ 0
+Text Notes 6000 4850 0    50   ~ 0
 I2C Expansion for\nDC/AC Current
 Text Notes 2550 700  0    50   ~ 0
@@
 NoConn ~ 9700 6000
 NoConn ~ 10150 6000
+$Comp
+L Device:CP1_Small C9
+U 1 1 62426391
+P 6550 6450
+F 0 "C9" H 6641 6496 50  0000 L CNN
+F 1 "180uF" H 6641 6405 50  0000 L CNN
+F 2 "Capacitor_SMD:CP_Elec_6.3x5.9" H 6550 6450 50  0001 C CNN
+F 3 "~" H 6550 6450 50  0001 C CNN
+F 4 "United Chemi-Con" H 6550 6450 50  0001 C CNN "Mfg"
+F 5 "APXN100ARA181MF61G" H 6550 6450 50  0001 C CNN "Mfg PN"
+	1    6550 6450
+	1    0    0    -1
+$EndComp
+$Comp
+L Device:R_Small R28
+U 1 1 6242951F
+P 6800 4250
+F 0 "R28" H 6859 4296 50  0000 L CNN
+F 1 "4.7k-DNP" H 6859 4205 50  0000 L CNN
+F 2 "Resistor_SMD:R_0805_2012Metric" H 6800 4250 50  0001 C CNN
+F 3 "~" H 6800 4250 50  0001 C CNN
+	1    6800 4250
+	1    0    0    -1
+$EndComp
+$Comp
+L Device:R_Small R27
+U 1 1 62442DA4
+P 7300 4250
+F 0 "R27" H 7359 4296 50  0000 L CNN
+F 1 "4.7k-DNP" H 7359 4205 50  0000 L CNN
+F 2 "Resistor_SMD:R_0805_2012Metric" H 7300 4250 50  0001 C CNN
+F 3 "~" H 7300 4250 50  0001 C CNN
+	1    7300 4250
+	1    0    0    -1
+$EndComp
+$Comp
+L power:+3.3V #PWR0132
+U 1 1 62443B09
+P 6800 4150
+F 0 "#PWR0132" H 6800 4000 50  0001 C CNN
+F 1 "+3.3V" H 6815 4323 50  0000 C CNN
+F 2 "" H 6800 4150 50  0001 C CNN
+F 3 "" H 6800 4150 50  0001 C CNN
+	1    6800 4150
+	1    0    0    -1
+$EndComp
+Wire Wire Line
+	6800 4350 6800 4450
+Connection ~ 6800 4450
+Wire Wire Line
+	6800 4450 7750 4450
+Wire Wire Line
+	7300 4350 7300 4550
+Connection ~ 7300 4550
+Wire Wire Line
+	7300 4550 7850 4550
+$Comp
+L power:+3.3V #PWR0133
+U 1 1 624CEE78
+P 7300 4150
+F 0 "#PWR0133" H 7300 4000 50  0001 C CNN
+F 1 "+3.3V" H 7315 4323 50  0000 C CNN
+F 2 "" H 7300 4150 50  0001 C CNN
+F 3 "" H 7300 4150 50  0001 C CNN
+	1    7300 4150
+	1    0    0    -1
+$EndComp
 $EndSCHEMATC

Commit message: layout P1.1 update U1 footprint to have 0.3mm vias
Parts:
- U1: footprint Package_SO:MSOP-8-1EP_3x3mm_P0.65mm_EP1.73x1.85mm_ThermalVias -> mate-net-monitor-special:MSOP-8-1EP_3x3mm_P0.65mm_EP1.88x2mm_ThermalVias0.3mm
Changed lines of the file:
@@
 F 0 "U1" H 2250 6767 50  0000 C CNN
 F 1 "LM5085MY" H 2250 6676 50  0000 C CNN
-F 2 "Package_SO:MSOP-8-1EP_3x3mm_P0.65mm_EP1.73x1.85mm_ThermalVias" H 2300 5750 50  0001 L CIN
+F 2 "mate-net-monitor-special:MSOP-8-1EP_3x3mm_P0.65mm_EP1.88x2mm_ThermalVias0.3mm" H 2300 5750 50  0001 L CIN
 F 3 "https://www.ti.com/lit/ds/symlink/lm5085.pdf" H 2250 6200 50  0001 C CNN
 	1    2250 6200
