File: pcb/mate-net-monitor.kicad_sch (KiCad schematic)
At the start: 66 parts, among them J1 6P6C, J2 6P6C, J3 Conn_02x02_Odd_Even, J4 Conn_01x08, J5 RJHSE-5081, Q1 Si2337DS, U1 LM5085MY, U2 TLP185, U3 TLP185, U4 TLP185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

Commit message: sch notes and cleanup
Parts:
- C1, C2: Mfg (none) -> TDK; Mfg PN (none) -> C3225X7S2A335K200AB

Commit message: mag net test rework and fw
Other:
- note added: "Rework: on Boron RX->D5 TX->D4"
- note added: "Rework: on baseboard U5.3 cut and connected to PB_D3 R23=100k"
- note added: "Rework: on baseboard replaced with Pololu D24V5F5 from R14/D5 to C6"
Changed lines of the file:
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@@
     (effects (font (size 1.27 1.27)) (justify left bottom))
+  )
+  (text "Rework:\non Boron\nRX->D5\nTX->D4" (at 191.135 67.31 0)
+    (effects (font (size 1.27 1.27) (thickness 0.254) bold) (justify left bottom))
   )
   (text "1.1mA\n@ 14V" (at 212.09 26.67 0)
@@
   (text "MATE Net\nUART @ Vbatt\n9600 9n1" (at 48.26 118.11 0)
     (effects (font (size 1.27 1.27)) (justify left bottom))
+  )
+  (text "Rework:\non baseboard\n\nU5.3 cut and\nconnected to\nPB_D3\n\nR23=100k"
+    (at 207.01 130.81 0)
+    (effects (font (size 1.27 1.27) (thickness 0.254) bold) (justify left bottom))
   )
   (text "1.1mA\n@ 56V\nlimiting\n" (at 76.2 29.21 0)
@@
     (effects (font (size 1.27 1.27)) (justify left bottom))
   )
+  (text "Rework:\non baseboard\n\nreplaced with Pololu D24V5F5\nfrom R14/D5 to C6"
+    (at 100.965 138.43 0)
+    (effects (font (size 1.27 1.27) (thickness 0.254) bold) (justify left bottom))
+  )
   (text "1.1mA\n@ 3.3V" (at 226.06 26.67 0)
