File: pcb-max3100-uart-adpt/max3100-uart-adpt.kicad_pcb (KiCad board)
At the start: 2 copper layers, 17.2 x 18 mm, 14 parts, among them IC1 MAX3100EEE+, J1 Conn_01x02, J2 Conn_01x06, J3 Conn_01x04, Q1 Q_NMOS_DUAL, Y1 3.6864MHz

Commit message: add pcb-max3100-uart-adpt gerbers
Changed lines of the file:
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@@
     (fp_line (start 1 -0.625) (end -1 -0.625) (layer "B.Fab") (width 0.1))
     (fp_line (start -1 -0.625) (end -1 0.625) (layer "B.Fab") (width 0.1))
-    (pad "1" smd roundrect (at -0.9125 0 270) (size 1.025 1.4) (layers "B.Cu" "B.Paste" "B.Mask") (roundrect_rratio 0.243902)
+    (pad "1" smd roundrect (at -0.9125 0 270) (size 1.025 1.4) (layers "B.Cu" "B.Paste" "B.Mask") (roundrect_rratio 0.243902439)
       (net 1 "+3V3") (pintype "passive"))
-    (pad "2" smd roundrect (at 0.9125 0 270) (size 1.025 1.4) (layers "B.Cu" "B.Paste" "B.Mask") (roundrect_rratio 0.243902)
+    (pad "2" smd roundrect (at 0.9125 0 270) (size 1.025 1.4) (layers "B.Cu" "B.Paste" "B.Mask") (roundrect_rratio 0.243902439)
       (net 19 "/UART_RXD") (pintype "passive"))
     (model "${KICAD6_3DMODEL_DIR}/Resistor_SMD.3dshapes/R_0805_2012Metric.wrl"
@@
     (fp_line (start 1 0.625) (end 1 -0.625) (layer "B.Fab") (width 0.1))
     (fp_line (start 1 -0.625) (end -1 -0.625) (layer "B.Fab") (width 0.1))
-    (pad "1" smd roundrect (at -0.9125 0 90) (size 1.025 1.4) (layers "B.Cu" "B.Paste" "B.Mask") (roundrect_rratio 0.243902)
+    (pad "1" smd roundrect (at -0.9125 0 90) (size 1.025 1.4) (layers "B.Cu" "B.Paste" "B.Mask") (roundrect_rratio 0.243902439)
       (net 20 "/UART_TXD") (pintype "passive"))
-    (pad "2" smd roundrect (at 0.9125 0 90) (size 1.025 1.4) (layers "B.Cu" "B.Paste" "B.Mask") (roundrect_rratio 0.243902)
+    (pad "2" smd roundrect (at 0.9125 0 90) (size 1.025 1.4) (layers "B.Cu" "B.Paste" "B.Mask") (roundrect_rratio 0.243902439)
       (net 24 "/UART_TXD_R") (pintype "passive"))
     (model "${KICAD6_3DMODEL_DIR}/Resistor_SMD.3dshapes/R_0805_2012Metric.wrl"
