File: pcb-max3100-uart-adpt/max3100-uart-adpt.kicad_sch (KiCad schematic)
At the start: 13 parts, among them IC1 MAX3100EEE+, J1 Conn_01x02, J2 Conn_01x06, J3 Conn_01x04, Q1 Q_NMOS_DUAL, Y1 3.6864MHz

Commit message: add pcb-max3100-uart-adpt gerbers
Parts:
- Q1: Mfg (none) -> Diodes Inc; Mfg PN (none) -> DMN5L06DMK-7
- RN1: value 1k -> 2.2k; Mfg (none) -> Yageo; Mfg PN (none) -> YC164-JR-072K2L
- Y1: Mfg (none) -> Abracon LLC; Mfg 2 (none) -> ECS Inc.; Mfg 2 PN (none) -> ECS-CTP-3.68-30-TR; Mfg PN (none) -> AWSCR-3.68CPLA-C30-T4
Changed lines of the file:
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@@
       (effects (font (size 1.27 1.27)) (justify left))
     )
-    (property "Value" "1k" (id 1) (at 181.61 147.3199 0)
+    (property "Value" "2.2k" (id 1) (at 181.61 147.3199 0)
       (effects (font (size 1.27 1.27)) (justify left))
     )
@@
     )
     (property "Datasheet" "" (id 3) (at 179.07 146.05 0)
+      (effects (font (size 1.27 1.27)) hide)
+    )
+    (property "Mfg" "Yageo" (id 4) (at 158.75 146.05 0)
+      (effects (font (size 1.27 1.27)) hide)
+    )
+    (property "Mfg PN" "YC164-JR-072K2L " (id 5) (at 158.75 146.05 0)
       (effects (font (size 1.27 1.27)) hide)
     )
@@
       (effects (font (size 1.27 1.27)) (justify left))
     )
-    (property "Value" "1k" (id 1) (at 161.29 147.3199 0)
+    (property "Value" "2.2k" (id 1) (at 161.29 147.3199 0)
       (effects (font (size 1.27 1.27)) (justify left))
     )
@@
     )
     (property "Datasheet" "" (id 3) (at 158.75 146.05 0)
+      (effects (font (size 1.27 1.27)) hide)
+    )
+    (property "Mfg" "Yageo" (id 4) (at 158.75 146.05 0)
+      (effects (font (size 1.27 1.27)) hide)
+    )
+    (property "Mfg PN" "YC164-JR-072K2L " (id 5) (at 158.75 146.05 0)
       (effects (font (size 1.27 1.27)) hide)
     )
@@
     )
     (property "Datasheet" "" (id 3) (at 134.62 165.1 0))
+    (property "Mfg" "Diodes Inc" (id 4) (at 93.98 165.1 0)
+      (effects (font (size 1.27 1.27)) hide)
+    )
+    (property "Mfg PN" "DMN5L06DMK-7" (id 5) (at 93.98 165.1 0)
+      (effects (font (size 1.27 1.27)) hide)
+    )
     (pin "1")
     (pin "2")
@@
     )
     (property "Datasheet" "" (id 3) (at 93.98 165.1 0))
+    (property "Mfg" "Diodes Inc" (id 4) (at 93.98 165.1 0)
+      (effects (font (size 1.27 1.27)) hide)
+    )
+    (property "Mfg PN" "DMN5L06DMK-7" (id 5) (at 93.98 165.1 0)
+      (effects (font (size 1.27 1.27)) hide)
+    )
     (pin "1")
     (pin "2")
@@
       (effects (font (size 1.27 1.27)) (justify left))
     )
-    (property "Value" "1k" (id 1) (at 99.06 147.3199 0)
+    (property "Value" "2.2k" (id 1) (at 99.06 147.3199 0)
       (effects (font (size 1.27 1.27)) (justify left))
     )
@@
     )
     (property "Datasheet" "" (id 3) (at 96.52 146.05 0)
+      (effects (font (size 1.27 1.27)) hide)
+    )
+    (property "Mfg" "Yageo" (id 4) (at 158.75 146.05 0)
+      (effects (font (size 1.27 1.27)) hide)
+    )
+    (property "Mfg PN" "YC164-JR-072K2L " (id 5) (at 158.75 146.05 0)
       (effects (font (size 1.27 1.27)) hide)
     )
@@
       (effects (font (size 1.27 1.27)) hide)
     )
+    (property "Mfg" "Abracon LLC" (id 4) (at 196.85 90.17 0)
+      (effects (font (size 1.27 1.27)) hide)
+    )
+    (property "Mfg PN" "AWSCR-3.68CPLA-C30-T4" (id 5) (at 196.85 90.17 0)
+      (effects (font (size 1.27 1.27)) hide)
+    )
+    (property "Mfg 2" "ECS Inc." (id 6) (at 196.85 90.17 0)
+      (effects (font (size 1.27 1.27)) hide)
+    )
+    (property "Mfg 2 PN" " ECS-CTP-3.68-30-TR" (id 7) (at 196.85 90.17 0)
+      (effects (font (size 1.27 1.27)) hide)
+    )
     (pin "1")
     (pin "2")
@@
       (effects (font (size 1.27 1.27)) (justify left))
     )
-    (property "Value" "1k" (id 1) (at 139.7 147.3199 0)
+    (property "Value" "2.2k" (id 1) (at 139.7 147.3199 0)
       (effects (font (size 1.27 1.27)) (justify left))
     )
@@
     )
     (property "Datasheet" "" (id 3) (at 137.16 146.05 0)
+      (effects (font (size 1.27 1.27)) hide)
+    )
+    (property "Mfg" "Yageo" (id 4) (at 158.75 146.05 0)
+      (effects (font (size 1.27 1.27)) hide)
+    )
+    (property "Mfg PN" "YC164-JR-072K2L " (id 5) (at 158.75 146.05 0)
       (effects (font (size 1.27 1.27)) hide)
     )
@@
     )
     (path "/2979bf79-00f8-477e-b1e5-27a50ae5be3e"
-      (reference "RN1") (unit 1) (value "1k") (footprint "Resistor_SMD:R_Array_Convex_4x0603")
+      (reference "RN1") (unit 1) (value "2.2k") (footprint "Resistor_SMD:R_Array_Convex_4x0603")
     )
     (path "/8ec704a2-e1ff-4f52-b99d-1043159f0f38"
-      (reference "RN1") (unit 2) (value "1k") (footprint "Resistor_SMD:R_Array_Convex_4x0603")
+      (reference "RN1") (unit 2) (value "2.2k") (footprint "Resistor_SMD:R_Array_Convex_4x0603")
     )
     (path "/b239e847-ac1a-498d-95ae-b2b8c2be1870"
-      (reference "RN1") (unit 3) (value "1k") (footprint "Resistor_SMD:R_Array_Convex_4x0603")
+      (reference "RN1") (unit 3) (value "2.2k") (footprint "Resistor_SMD:R_Array_Convex_4x0603")
     )
     (path "/16ba8ee6-0c51-4bb5-8b3f-a1ee9395a514"
-      (reference "RN1") (unit 4) (value "1k") (footprint "Resistor_SMD:R_Array_Convex_4x0603")
+      (reference "RN1") (unit 4) (value "2.2k") (footprint "Resistor_SMD:R_Array_Convex_4x0603")
     )
     (path "/8f7d967f-4648-4a5a-bd7e-58b298eaf68c"
